Commit message: Imu link changed

File: husky_description/urdf/husky.urdf.xacro (robot description, xacro)
@@ -98,11 +98,11 @@
   <!-- IMU Link is the standard mounting position for the UM6 IMU.-->
   <!-- Can be modified with environment variables in /etc/ros/setup.bash -->
-  <link name="imu_link"/>
+  <link name="zed_imu_link"/>
   <joint name="imu_joint" type="fixed">
     <origin xyz="$(optenv HUSKY_IMU_XYZ 0.19 0 0.149)" rpy="$(optenv HUSKY_IMU_RPY 0 -1.5708 3.1416)" />
     <parent link="base_link" />
-    <child link="imu_link" />
+    <child link="zed_imu_link" />
   </joint>
-  <gazebo reference="imu_link">
+  <gazebo reference="zed_imu_link">
   </gazebo>
   <!-- Husky wheel macros -->
